File: raspi/raspi-avr-teletext-2side.sch (EAGLE design)
At the start: 17 parts, among them U1 ATMEGA328P, U2 EL1883, X1 WBTOR1

Commit message: Fix MOSI/MISO
I can never remember whether you are supposed to flip these or not.
Connections:
- net MISO: now also D1.21-SPI-MISO; no longer D1.19-SPI-MOSI
- net MOSI: now also D1.19-SPI-MOSI; no longer D1.21-SPI-MISO
Changed lines of the file:
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@@
 <setting verticaltext="up"/>
 </settings>
-<grid distance="0.1" unitdist="inch" unit="inch" style="lines" multiple="1" display="no" altdistance="0.05" altunitdist="inch" altunit="inch"/>
+<grid distance="0.1" unitdist="inch" unit="inch" style="lines" multiple="1" display="no" altdistance="0.01" altunitdist="inch" altunit="inch"/>
 <layers>
 <layer number="1" name="Top" color="4" fill="1" visible="no" active="no"/>
@@
 </segment>
 <segment>
-<pinref part="D1" gate="G$1" pin="19-SPI-MOSI"/>
-<wire x1="152.4" y1="33.02" x2="149.86" y2="33.02" width="0.1524" layer="91"/>
-<wire x1="149.86" y1="33.02" x2="144.78" y2="27.94" width="0.1524" layer="91"/>
-<wire x1="144.78" y1="27.94" x2="142.24" y2="27.94" width="0.1524" layer="91"/>
+<pinref part="D1" gate="G$1" pin="21-SPI-MISO"/>
 <junction x="142.24" y="27.94"/>
 <label x="141.605" y="27.305" size="1.778" layer="95" rot="MR0"/>
+<wire x1="152.4" y1="27.94" x2="142.24" y2="27.94" width="0.1524" layer="91"/>
 </segment>
 </net>
@@
 </segment>
 <segment>
-<pinref part="D1" gate="G$1" pin="21-SPI-MISO"/>
-<wire x1="152.4" y1="27.94" x2="149.86" y2="27.94" width="0.1524" layer="91"/>
-<wire x1="149.86" y1="27.94" x2="144.78" y2="33.02" width="0.1524" layer="91"/>
-<wire x1="144.78" y1="33.02" x2="142.24" y2="33.02" width="0.1524" layer="91"/>
+<pinref part="D1" gate="G$1" pin="19-SPI-MOSI"/>
 <junction x="142.24" y="33.02"/>
 <label x="141.605" y="32.385" size="1.778" layer="95" rot="MR0"/>
-</segment>
-</net>
+<wire x1="152.4" y1="33.02" x2="142.24" y2="33.02" width="0.1524" layer="91"/>
+</segment>
+</net>
